Commit message: Updates

File: local_env/Robots/hermes_robot/urdf/hermes_robot.urdf (robot description, URDF)
Before this commit: robot Assem1.SLDASM, 9 links, 8 joints
Links:
- link Drive1: geometry collision mesh filename=package://hermes_robot/meshes/Drive1.STL; visual mesh filename=package://hermes_robot/meshes/Drive1.STL
- link Drive2: geometry collision mesh filename=package://hermes_robot/meshes/Drive2.STL; visual mesh filename=package://hermes_robot/meshes/Drive2.STL
- link Drive3: geometry collision mesh filename=package://hermes_robot/meshes/Drive3.STL; visual mesh filename=package://hermes_robot/meshes/Drive3.STL
- link Drive4: geometry collision mesh filename=package://hermes_robot/meshes/Drive4.STL; visual mesh filename=package://hermes_robot/meshes/Drive4.STL
- link Revolve1: geometry collision mesh filename=package://hermes_robot/meshes/Revolve1.STL; visual mesh filename=package://hermes_robot/meshes/Revolve1.STL
- link Revolve2: geometry collision mesh filename=package://hermes_robot/meshes/Revolve2.STL; visual mesh filename=package://hermes_robot/meshes/Revolve2.STL
- link Revolve3: geometry collision mesh filename=package://hermes_robot/meshes/Revolve3.STL; visual mesh filename=package://hermes_robot/meshes/Revolve3.STL
- link Revolve4: geometry collision mesh filename=package://hermes_robot/meshes/Revolve4.STL; visual mesh filename=package://hermes_robot/meshes/Revolve4.STL
- link base_link: geometry collision mesh filename=package://hermes_robot/meshes/base_link.STL; visual mesh filename=package://hermes_robot/meshes/base_link.STL
Joints:
- joint Drive1: limit lower=0 upper=0 effort=0 velocity=0 -> lower=0 upper=6.28 effort=0 velocity=0

Commit message: Updates to model. Now just need to fix coordinate frames for axis I think

File: local_env/Robots/hermes_robot/urdf/hermes_robot.urdf (robot description, URDF)
Before this commit: robot hermes_robot, 9 links, 8 joints
Links:
- link Drive1: mass 0.700310778907897 -> 0.968782085796601
- link Drive2: mass 0.700310778907893 -> 0.968781690098536
- link Drive3: mass 0.700310778907896 -> 0.968781681639634
- link Drive4: mass 0.700310778907897 -> 0.850687457270781
- link Revolve1: mass 0.22984858770233 -> 0.269967968577388
- link Revolve2: mass 0.229848600316094 -> 0.278169948732177
- link Revolve3: mass 0.229848603142654 -> 0.282156119775798
- link Revolve4: mass 0.229848600569597 -> 0.278169965817926
- link base_link: mass 0.469800963040705 -> 5.7729702362968
Joints:
- joint Drive1: axis 0.99884 -0.048238 0 -> 0.97870110149261 0.205290413651375 0; limit lower=0 upper=6.28 effort=0 velocity=0 -> lower=0 upper=0 effort=0 velocity=0; origin xyz=0 0 -0.003175 rpy=0 0 3.1416 -> xyz=0 0 0 rpy=0 0 0; type revolute -> continuous
- joint Drive2: axis 1 0.002809 0 -> -0.99999 -0.0043624 0; origin xyz=0 0 -0.003175 rpy=0 0 3.1416 -> xyz=0 0 0 rpy=0 0 0; type revolute -> continuous
- joint Drive3: origin xyz=0 0 -0.003175 rpy=0 0 3.1416 -> xyz=0 0 0 rpy=0 0 0; type revolute -> continuous
- joint Drive4: axis 0.99999 0.0034092 0 -> 0.99632 0.085731 0; origin xyz=0 0 -0.003175 rpy=0 0 3.1416 -> xyz=0 0 0 rpy=0 0 0; type revolute -> continuous
- joint Revolve1: origin xyz=0 0 -0.003175 rpy=0 0 3.1416 -> xyz=0 0 0 rpy=0 0 0; type revolute -> continuous
- joint Revolve2: origin xyz=0 0 -0.003175 rpy=0 0 3.1416 -> xyz=0 0 0 rpy=0 0 0; type revolute -> continuous
- joint Revolve3: origin xyz=0 0 -0.003175 rpy=0 0 3.1416 -> xyz=0 0 0 rpy=0 0 0; type revolute -> continuous
- joint Revolve4: origin xyz=0 0 -0.003175 rpy=0 0 3.1416 -> xyz=0 0 0 rpy=0 0 0; type revolute -> continuous

Commit message: Working Gazebo World Deployer

File: local_env/Robots/hermes_robot/urdf/hermes_robot.urdf (robot description, URDF)
Before this commit: robot hermes_robot, 9 links, 8 joints
Links:
- link Drive1: mass 0.968782085796601 -> 0.968781681350828
- link Drive2: mass 0.968781690098536 -> 0.968781685280355
- link Drive3: mass 0.968781681639634 -> 0.968781680813743
- link Drive4: mass 0.850687457270781 -> 0.850687527986548
- link Revolve1: mass 0.269967968577388 -> 0.269968020345209
- link Revolve2: mass 0.278169948732177 -> 0.278169943270248
- link Revolve3: mass 0.282156119775798 -> 0.282156111545984
- link Revolve4: mass 0.278169965817926 -> 0.278169949354846
Joints:
- removed joint Drive1
- removed joint Drive2
- removed joint Drive3
- removed joint Drive4
- removed joint Revolve1
- removed joint Revolve2
- removed joint Revolve3
- removed joint Revolve4
- added joint Joint_Drive1: type continuous, parent Revolve1, child Drive1, origin xyz=0.058211 -0.00088915 -0.23708 rpy=0 0 0, axis -0.99995 0.0098663 0, limit lower=0 upper=0 effort=0 velocity=10
- added joint Joint_Drive2: type continuous, parent Revolve2, child Drive2, origin xyz=0.061783 -0.00014808 -0.23708 rpy=0 0 0, axis 0.99997 -0.0074916 0, limit lower=0 upper=0 effort=0 velocity=10
- added joint Joint_Drive3: type continuous, parent Revolve3, child Drive3, origin xyz=-0.23708 -0.0003149 -0.061783 rpy=0 0 0, axis 0 -0.010191 -0.99995, limit lower=0 upper=0 effort=0 velocity=10
- added joint Joint_Drive4: type continuous, parent Revolve4, child Drive4, origin xyz=0.058218 8.492E-05 -0.23708 rpy=0 0 0, axis -0.99998 -0.0068655 0, limit lower=0 upper=0 effort=0 velocity=10
- added joint Joint_Revolve1: type continuous, parent base_link, child Revolve1, origin xyz=0.14293 0.16281 0.080887 rpy=0 0 0, axis 0 0 -1, limit lower=0 upper=6.28 effort=0 velocity=0
- added joint Joint_Revolve2: type continuous, parent base_link, child Revolve2, origin xyz=0.14237 -0.16281 0.080887 rpy=0 0 0, axis 0 0 -1, limit lower=0 upper=6.28 effort=0 velocity=0
- added joint Joint_Revolve3: type continuous, parent base_link, child Revolve3, origin xyz=-0.14293 -0.16281 0.080887 rpy=3.1416 -1.5708 0, axis -1 0 0, limit lower=0 upper=6.28 effort=0 velocity=0
- added joint Joint_Revolve4: type continuous, parent base_link, child Revolve4, origin xyz=-0.14237 0.16281 0.080887 rpy=0 0 0, axis 0 0 -1, limit lower=0 upper=6.28 effort=0 velocity=0
