Commit message: Better web controller, working visual synced from Gazebo to RVIZ

File: src/hermes_robot_description/urdf/hermes.urdf (robot description, URDF)
Before this commit: robot hermes_robot_description, 9 links, 8 joints
Links:
- added link CameraVision, mass 0.00122306679751053; collision mesh filename=package://hermes_robot_description/meshes/CameraVision.STL; visual mesh filename=package://hermes_robot_description/meshes/CameraVision.STL
- added link Camera_pivot, mass 1.28786623127725; collision mesh filename=package://hermes_robot_description/meshes/Camera_pivot.STL; visual mesh filename=package://hermes_robot_description/meshes/Camera_pivot.STL
Joints:
- added joint CameraVisionJoint: type fixed, parent Camera_pivot, child CameraVision, origin xyz=-0.0545 0.002307 -0.016859 rpy=3.1416 0 3.1416, axis 0 0 0
- added joint Joint_Camera_pivot: type revolute, parent base_link, child Camera_pivot, origin xyz=0.05435 0.23015 0.06 rpy=1.5708 0 0, axis 1 0 0, limit lower=0 upper=0 effort=0 velocity=0

Commit message: Better controller

File: src/hermes_robot_description/urdf/hermes.urdf (robot description, URDF)
Before this commit: robot hermes_robot_description, 11 links, 10 joints
Joints:
- joint Joint_Revolve1: limit lower=0 upper=6.28 effort=0 velocity=0 -> lower=-6.28 upper=6.28 effort=0 velocity=0
- joint Joint_Revolve2: limit lower=0 upper=6.28 effort=0 velocity=0 -> lower=-6.28 upper=6.28 effort=0 velocity=0
- joint Joint_Revolve3: limit lower=0 upper=6.28 effort=0 velocity=0 -> lower=-6.28 upper=6.28 effort=0 velocity=0
- joint Joint_Revolve4: limit lower=0 upper=6.28 effort=0 velocity=0 -> lower=-6.28 upper=6.28 effort=0 velocity=0

Commit message: Some updates to the URDF, transfering them to the SDF

File: src/hermes_robot_description/urdf/hermes.urdf (robot description, URDF)
Before this commit: robot hermes_robot_description, 12 links, 11 joints
Joints:
- joint Joint_Drive1: axis -0.99995 0.0098663 0 -> 1 0 0
- joint Joint_Drive2: axis 0.99997 -0.0074916 0 -> 1 0 0
- joint Joint_Drive3: axis 0 -0.010191 -0.99995 -> 1 0 0; origin xyz=-0.23708 -0.0003149 -0.061783 rpy=0 0 0 -> xyz=0.061783 -0.00014808 -0.23708 rpy=0 0 0
- joint Joint_Drive4: axis -0.99998 -0.0068655 0 -> 1 0 0
- joint Joint_Revolve3: axis -1 0 0 -> 0 0 -1; origin xyz=-0.14293 -0.16281 0.080887 rpy=3.1416 -1.5708 0 -> xyz=-0.14293 -0.16281 0.080887 rpy=0 0 0
