Commit message: Only managing a single urdf which is converted by the launch file into an SDF

File: src/hermes_robot_description/urdf/corrected.urdf (robot description, URDF)
Before this commit: robot hermes_robot_description, 13 links, 12 joints
Links:
- removed link depth_camera
Joints:
- removed joint depth_camera_joint
