Commit message: Updates to the position of the camera

File: src/hermes_robot_description/urdf/corrected.urdf.xacro (robot description, xacro)
@@ -635,6 +635,16 @@
     </sensor>
   </gazebo>
-  <gazebo reference="base_footprint">
+  <!-- Create a static link that connects to CameraVisionLink but is moved slighly -->
+  <link name="DepthCameraFrame">
+    <pose>0 0 0 0 0 0</pose> <!-- Offset and rotation -->
+  </link>
+  <joint name="DepthCameraJoint" type="fixed">
+    <origin rpy="0 -1.5708 0" />
+    <parent link="CameraVisionLink"/>
+    <child link="DepthCameraFrame"/>
+  </joint>
+  <gazebo reference="DepthCameraFrame">
     <sensor name="RealsenseD435" type="rgbd_camera">
+    <pose>0 0 0 0 0 0</pose>
       <camera>
         <horizontal_fov>1.25</horizontal_fov>
@@ -647,5 +657,5 @@
           <far>100</far>
         </clip>
-        <optical_frame_id>base_footprint</optical_frame_id>
+        <optical_frame_id>DepthCameraFrame</optical_frame_id>
       </camera>
       <update_rate>10</update_rate>
@@ -661,5 +671,5 @@
     <child link="front_realsense" />
   </joint> -->
-  <gazebo reference ="base_link">
+  <gazebo reference="base_link">
     <sensor name="imu" type="imu">
       <always_on>true</always_on>

Commit message: Updates on for mapping

File: src/hermes_robot_description/urdf/corrected.urdf.xacro (robot description, xacro)
@@ -637,8 +637,8 @@
   <!-- Create a static link that connects to CameraVisionLink but is moved slighly -->
   <link name="DepthCameraFrame">
-    <pose>0 0 0 0 0 0</pose> <!-- Offset and rotation -->
+    <pose>0 0 0 0 0 1.57</pose> <!-- Offset and rotation -->
   </link>
   <joint name="DepthCameraJoint" type="fixed">
-    <origin rpy="0 -1.5708 0" />
+    <origin rpy="-1.57 -1.57 0" />
     <parent link="CameraVisionLink"/>
     <child link="DepthCameraFrame"/>

Commit message: First draft, working Nav2

File: src/hermes_robot_description/urdf/corrected.urdf.xacro (robot description, xacro)
@@ -6,5 +6,5 @@
     <parent link="base_footprint" />
     <child link="base_link" />
-    <origin xyz="0 0 0" rpy="0 0 0" />
+    <origin xyz="0 0 .22" rpy="0 0 0" />
   </joint>
   <link name="base_footprint">
@@ -637,5 +637,5 @@
   <!-- Create a static link that connects to CameraVisionLink but is moved slighly -->
   <link name="DepthCameraFrame">
-    <pose>0 0 0 0 0 1.57</pose> <!-- Offset and rotation -->
+    <pose>0 0 0 0 0 0</pose> <!-- Offset and rotation -->
   </link>
   <joint name="DepthCameraJoint" type="fixed">
